File: eagle/lil_gate_sequencer.brd (EAGLE design)
At the start: 100 x 80 mm, 70 parts, among them IC1 4093N, IC2 4017N, Q1 2N3904, Q2 2N3904

Commit message: better routes and gcode
Parts:
- removed OUT_LED1: LSP11, solpad:LSP11
- C2: device rcl:B45181A -> rcl:B45181B
- OUT_LED: value LSP11 -> (none); device solpad:LSP11 -> led:LED5MM
- moved R1 8.39 mm to (95.0, 29.1)
- moved R13 6.48 mm to (2.54, 40.6), turned to 90 degrees
- moved C2 5.08 mm to (25.4, 62.2)
- moved R10 4.58 mm to (3.81, 29.2), turned to 0 degrees
- moved FB1 3.81 mm to (19.1, 57.1)
- moved C3 2.69 mm to (48.6, 55.9)
- moved Q1 2.54 mm to (73.7, 66.0)
- moved R3 2.54 mm to (78.7, 66.0)
- moved R7 1.80 mm to (54.6, 69.8)
- moved LENGTH_1 1.80 mm to (19.1, 73.7)
- moved JP1 1.80 mm to (7.62, 72.4), turned to 0 degrees
- moved C6 1.27 mm to (63.5, 73.7)
- moved C4 1.27 mm to (24.1, 74.9)
- moved ENABLE_2 1.27 mm to (27.9, 74.9)
- moved R11 1.27 mm to (22.9, 69.8)
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Connections:
- net N$43: now also OUT_LED.K; no longer OUT_LED1.MP
- net N$6: now also OUT_LED.A; no longer OUT_LED.MP
Routing:
- net N$35: track 4.86 -> 120.1 mm
- net N$15: track 3.07 -> 56.0 mm
- net N$23: track 3.07 -> 54.5 mm, vias 0 -> 2
- net N$33: track 3.07 -> 52.8 mm
- net N$17: track 3.07 -> 46.1 mm
- net N$21: track 3.70 -> 46.4 mm, vias 0 -> 2
- net N$19: track 3.07 -> 43.4 mm
- net N$31: track 3.07 -> 34.1 mm
- net N$29: track 3.07 -> 24.3 mm
- net N$25: track 3.07 -> 21.6 mm, vias 0 -> 2
- net N$27: track 3.07 -> 20.8 mm
- net N$4: track 30.2 -> 47.3 mm
- net N$6: track 93.9 -> 78.7 mm, vias 2 -> 0
- net N$7: track 18.0 -> 9.61 mm
- net GND: track 435.6 -> 440.9 mm, vias 2 -> 4
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